File: Hardware/prot2/Eagle/colecovision2.brd (EAGLE design)
At the start: 73.6 x 89.8 mm, 26 parts, among them IC1 CY7C1019CV33-12VC

Commit message: CTRL+ALT+BACKSPACE works! Multcart needs 8K RAM, then updated TOPs for supply 8K for Multcart and 1K for games. Tested. Sigma-delta DAC works better with resistor 2K2 and capacitor 10n. Updated prot2 eagle project and related files.
Parts:
- C3: value 4n7 -> 10n
- R1: value 3K3 -> 2K2
Changed lines of the file:
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@@
 <attribute name="VALUE" x="34.925" y="73.025" size="1.778" layer="27" ratio="10" rot="R180"/>
 </element>
-<element name="C3" library="rcl" package="C1206" value="4n7" x="8.255" y="76.2" smashed="yes" rot="MR0">
+<element name="C3" library="rcl" package="C1206" value="10n" x="8.255" y="76.2" smashed="yes" rot="MR0">
 <attribute name="NAME" x="5.08" y="75.565" size="1.27" layer="26" rot="MR0"/>
 <attribute name="VALUE" x="13.97" y="75.565" size="1.27" layer="28" rot="MR0"/>
 </element>
-<element name="R1" library="rcl" package="R1206" value="3K3" x="8.255" y="73.66" smashed="yes" rot="MR180">
+<element name="R1" library="rcl" package="R1206" value="2K2" x="8.255" y="73.66" smashed="yes" rot="MR180">
 <attribute name="NAME" x="3.175" y="74.295" size="1.27" layer="26" rot="MR180"/>
 <attribute name="VALUE" x="11.43" y="74.295" size="1.27" layer="28" rot="MR180"/>
