File: Hardware/prot2/Eagle/colecovision2.sch (EAGLE design)
At the start: 26 parts, among them IC1 CY7C1019CV33-12VC

Commit message: CTRL+ALT+BACKSPACE works! Multcart needs 8K RAM, then updated TOPs for supply 8K for Multcart and 1K for games. Tested. Sigma-delta DAC works better with resistor 2K2 and capacitor 10n. Updated prot2 eagle project and related files.
Parts:
- C3: value 4n7 -> 10n
- R1: value 3K3 -> 2K2
Changed lines of the file:
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@@
 <part name="GND4" library="supply1" deviceset="GND" device=""/>
 <part name="X3" library="fabio" deviceset="VGA" device="H"/>
-<part name="C3" library="rcl" deviceset="C-EU" device="C1206" value="4n7"/>
-<part name="R1" library="rcl" deviceset="R-EU_" device="R1206" value="3K3"/>
+<part name="C3" library="rcl" deviceset="C-EU" device="C1206" value="10n"/>
+<part name="R1" library="rcl" deviceset="R-EU_" device="R1206" value="2K2"/>
 <part name="R2" library="rcl" deviceset="R-EU_" device="R1206" value="4K"/>
 <part name="R3" library="rcl" deviceset="R-EU_" device="R1206" value="2K"/>
